File: FE_channel.kicad_sch (KiCad schematic)
At the start: 29 parts, among them J1 731000105, K1 UD2-4.5NUN-L, K2 UD2-4.5NUN-L, Q1 DMN61D8LQ, Q2 DMN61D8LQ

Commit message: finished the FE channel and voltage generation
Parts:
- removed J1: 731000105, 731000105:CONN_73100-0105_MOL, symbol 731000105:731000105
- removed K1, K2: UD2-4.5NUN-L, UD2-4.5NUN-L:RELAY_UD2-4.5NUN-L, symbol UD2-4.5NUN-L:UD2-4.5NUN-L_seperated
- added C11: 1pF, Capacitor_SMD:C_0805_2012Metric_Pad1.18x1.45mm_HandSolder, symbol Device:C
- added C12: 8pF, Capacitor_SMD:C_0805_2012Metric_Pad1.18x1.45mm_HandSolder, symbol Device:C
- added C13: 3pF, Capacitor_SMD:C_0805_2012Metric_Pad1.18x1.45mm_HandSolder, symbol Device:C
- added C14, C41, C42, C43: 100nF, Capacitor_SMD:C_0805_2012Metric_Pad1.18x1.45mm_HandSolder, symbol Device:C
- added C15: 1nF, Capacitor_SMD:C_0805_2012Metric_Pad1.18x1.45mm_HandSolder, symbol Device:C
- added C16: 10nF, Capacitor_SMD:C_0805_2012Metric_Pad1.18x1.45mm_HandSolder, symbol Device:C
- added C17, C18, C20: 100pF, Capacitor_SMD:C_0805_2012Metric_Pad1.18x1.45mm_HandSolder, symbol Device:C
- added C19: 68pF, Capacitor_SMD:C_0805_2012Metric_Pad1.18x1.45mm_HandSolder, symbol Device:C
- added C21, C22, C23, C24, C25, C26, C44, C45: 10uF, Capacitor_SMD:C_0805_2012Metric_Pad1.18x1.45mm_HandSolder, symbol Device:C
- added C27, C28, C29, C30, C31, C32, C33, C34, C35, C36, C37, C38, C39, C46, C47, C48, C49: 1uF, Capacitor_SMD:C_0805_2012Metric_Pad1.18x1.45mm_HandSolder, symbol Device:C
- added C40: 2-6pF, Thunderscope_Rev5:EW_TRIMCAP, symbol Thunderscope_Rev5:CAP TRIMMER 2-6PF 100V
- added FB1, FB2: 120@100MHZ, Inductor_SMD:L_0805_2012Metric_Pad1.05x1.20mm_HandSolder, symbol Device:FerriteBead
- added J2: BNC, Thunderscope_Rev5:MOL_0731000105, symbol Thunderscope_Rev5:BNC JACK R/A
- added K1, K3: UD2-4.5NUN-L, Thunderscope_Rev5:KEMET_UD2-4.5NUN-L, symbol Thunderscope_Rev5:RELAY DPDT-NO UD2-4.5NUN-L
- added R25, R46, R47: 0R, Resistor_SMD:R_0805_2012Metric_Pad1.20x1.40mm_HandSolder, symbol Device:R
- added R26, R43, R44: 1K, Resistor_SMD:R_0805_2012Metric_Pad1.20x1.40mm_HandSolder, symbol Device:R
- added R27, R28: 976K, Resistor_SMD:R_0805_2012Metric_Pad1.20x1.40mm_HandSolder, symbol Device:R
- added R29: 20K, Resistor_SMD:R_0805_2012Metric_Pad1.20x1.40mm_HandSolder, symbol Device:R
- added R30: 909K, Resistor_SMD:R_0805_2012Metric_Pad1.20x1.40mm_HandSolder, symbol Device:R
- added R31: 30R, Resistor_SMD:R_0805_2012Metric_Pad1.20x1.40mm_HandSolder, symbol Device:R
- added R32, R38, R40: 90.9K, Resistor_SMD:R_0805_2012Metric_Pad1.20x1.40mm_HandSolder, symbol Device:R
- added R33, R39, R45: 10K, Resistor_SMD:R_0805_2012Metric_Pad1.20x1.40mm_HandSolder, symbol Device:R
- added R34, R36: 10M, Resistor_SMD:R_0805_2012Metric_Pad1.20x1.40mm_HandSolder, symbol Device:R
- added R35: 2K, Resistor_SMD:R_0805_2012Metric_Pad1.20x1.40mm_HandSolder, symbol Device:R
- added R37: 35.7K, Resistor_SMD:R_0805_2012Metric_Pad1.20x1.40mm_HandSolder, symbol Device:R
- added R41: 2K TRIMPOT, Thunderscope_Rev5:BOU_3mm_POT, symbol Thunderscope_Rev5:TRIMMER 2K OHM 0.1W J LEAD TOP
- added R42: 49.9K, Resistor_SMD:R_0805_2012Metric_Pad1.20x1.40mm_HandSolder, symbol Device:R
- added TP3, TP4, TP5: TestPoint, TestPoint:TestPoint_Pad_D2.0mm, symbol Connector:TestPoint
- added U3: TMUX4053, Thunderscope_Rev5:TI_TSOT-23-16_DYY0016A, symbol Thunderscope_Rev5:IC SWITCH 3X SPDT TMUX4053
- added U4: OPA140AIDBVR, Thunderscope_Rev5:GEN_SOT23_5_950_2900X1600X1450, symbol Thunderscope_Rev5:IC OPAMP OPA140
- added U5: BUF802, Thunderscope_Rev5:TI_VQFN_RGT0016C, symbol Thunderscope_Rev5:IC BUFFER AMP BUF802
- added U6: LMH6518, Thunderscope_Rev5:TI_WQFN_RGH0016A, symbol Thunderscope_Rev5:IC PGA LMH6518
- C1: value C -> 18pF
- C2, C3: value C -> 3pF
- C4: value C -> 0.3pF
- R17: value R -> 30R
- R18: value R -> 15R
- TP1, TP2: footprint (none) -> TestPoint:TestPoint_Pad_D2.0mm
Connections:
- net +5V: now also C21.2, C22.2, C23.2, C27.2, C28.2, C29.2, C30.2, C31.2, C32.2, C39.2, C44.2, FB2.1, U3.16 (VDD), U4.5 (V+), U5.1 (Vs+), U5.12 (Vso+), U5.15 (CLH)
- net ATTEN_IN: now also K1.3, K3.6
- net ATTEN_OUT: now also K1.6, R30.2, R31.1
- net BNC_IN: now also J2.1 (Signal), K3.3
- net GND: now also C2.1, C12.2, C13.2, C14.1, C20.1, C21.1, C22.1, C23.1, C24.2, C25.2, C26.2, C27.1, C28.1, C29.1, C30.1, C31.1, C32.1, C33.2, C34.2, C35.2, C36.2, C37.2, C38.2, C39.1, C40.2, C41.1, C42.1, C43.1, C44.1, C45.1, C46.1, C47.1, C48.1, C49.1, J2.2 (SHIELD), R29.2, R32.1, R33.1, R34.1, R41.3, U3.6 (~{EN}), U3.8 (GND), U5.14 (CLL), U5.17 (PAD), U6.17 (PAD), U6.5 (GND), U6.8 (GND); no longer C1.2, C3.2
- net TERM: no longer R23.2, R24.1, TP2.1
- net at C6.1, C7.1, D1.1 (K)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: now also K3.1
- net at D1.2 (A), Q1.3 (D): now also K3.8
- net at R17.2: now also R16.1, K3.7; no longer C2.1
- net TERM_50Z: now reaches R15.1, R18.1
- net TERM_50Z: now also C1.1, K3.4; no longer C3.1, C4.2
- net at C4.1: now also R28.2; no longer R18.2
- net at C10.1, C9.1, D2.1 (K)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: now also K1.1
- net at D2.2 (A), Q2.3 (D): now also K1.8
- new net: R37.2, U5.7 (R_Bias)
- new net: C17.2, R35.1, U3.4 (D3), U4.1 (OUT)
- new net: C16.1, R30.1, R32.2, U3.14 (D1)
- new net: C16.2, R34.2, U3.13 (S1B), U4.3 (+)
- new net: C2.2, R26.1
- new net: R47.2, U6.14 (OUT_N)
- new net: R46.2, U6.15 (OUT_P)
- new net: R39.1, R41.1, R41.2
- new net: R38.1, R39.2, R40.2
- new net: C15.1, R31.2
- new net: C19.1, U3.1 (S2B)
- new net: C18.1, U3.2 (S2A)
- new net: C19.2, U3.3 (S3B)
- new net: C18.2, U3.5 (S3A)
- new net: C11.2, C12.1, C3.1, R28.1
- new net: C1.2, R25.1
- new net +3V3_PGA: C49.2, R45.2, U6.12 (VDD)
- new net +VPGA: C45.2, C46.2, C47.2, C48.2, FB2.2, U6.3 (VCC), U6.4 (VCC)
- new net -5V: C24.1, C25.1, C26.1, C33.1, C34.1, C35.1, C36.1, C37.1, C38.1, R37.1, U3.7 (VSS), U4.2 (V-), U5.10 (Vso-), U5.5 (Vs-), U5.6 (Aux_Bias), U5.8 (Vs-)
- new net -VBIAS: C14.2, C41.2, R40.1, R43.2, R44.2
- new net ATTEN: R23.2, R24.1, TP2.1
- new net ATTEN_1X: K1.4, K1.5
- new net ATTEN_50X_IN: C3.2, C4.2, K1.2, R26.2, R27.2
- new net ATTEN_50X_OUT: C11.1, C13.1, C40.1, K1.7, R27.1, R29.1
- new net BUF_IN: C15.2, R36.1, U5.2 (IN)
- new net BUF_IN_AUX: C20.2, R35.2, U5.4 (IN_Aux)
- new net BUF_IN_BIAS: R36.2, U5.3 (IN_Bias)
- new net BUF_OUT: R38.2, R42.2, U5.11 (OUT)
- new net BUF_OUT_R: R42.1, U6.6 (IN_P)
- new net DC_CPL: R33.2, TP3.1, U3.10 (SEL2), U3.11 (SEL1), U3.9 (SEL3)
- new net DC_FB: C17.1, U3.15 (D2), U4.4 (-)
- new net OUT_N: R47.1
- new net OUT_P: R46.1
- new net PGA_BIAS: C43.2, FB1.2, R43.1, R44.1, TP4.1, U6.7 (IN_N)
- new net PGA_CSn: R45.1, TP5.1, U6.9 (CSn)
- new net PGA_SCLK: U6.11 (SCLK)
- new net PGA_SDIO: U6.10 (SDIO)
- new net TERM_1M: K3.2, R17.1
- new net TERM_50Z_R: K3.5, R18.2, R25.2
- new net TRIM: C42.2, FB1.1
- new net VCM: U6.13 (VCM)
- no-connect marks 0 -> 4
Other:
- note added: "(NOTE: this was just copy pasted from the og project. need to reverify)"
- note added: "100k R_Bias wil be lower: 17mA per rail was measured on the EVM"
- note added: "Input Buffer and AC/DC Coupling"
- note added: "Max VCC current after configuration turns off AUX output: 0.165A"
- note added: "Max VCC current before configuration (AUX output on): 0.225A"
- note added: "Max VDD current: 0.35mA"
- note added: "Max current for 35.7kOhm R_Bias: 24mA @ V+ and 24mA @ V-"
- note added: "Programmable Gain Amplifier"
- note added: "Termination and Attenuation"
- note added: "This cap is switched in during AC coupling"
- note added: "This cap is switched in during DC coupling"
- note removed: "1MZ path"
- note removed: "1x Attenuation"
- note removed: "50Z path"
- note removed: "50x Attenuation"
- note removed: "fine tuning circuitry"
- moved on the sheet: C10, C5, C6, C7, C8, C9, D1, D2, Q1, Q2, R15, R16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

Commit message: updated the resistor sizings from all 0805 to 0402, 0603 and 0805s, to match the thunderscope directly
Parts:
- removed Q1, Q2: DMN61D8LQ, Package_TO_SOT_SMD:SOT-23, symbol Transistor_FET:DMN61D8LQ
- added Q1, Q5: DMN62D0UW, Thunderscope_Rev5:GEN_SOT_323, symbol Thunderscope_Rev5:NMOS DMN62D0UW
- C1, C10, C11, C12, C13, C14, C17, C18, C19, C2, C20, C27, C28, C29, C3, C30, C31, C32, C33, C34, C35, C36, C37, C38, C39, C4, C41, C42, C43, C46, C47, C48, C49, C7: footprint Capacitor_SMD:C_0805_2012Metric_Pad1.18x1.45mm_HandSolder -> Capacitor_SMD:C_0402_1005Metric_Pad0.74x0.62mm_HandSolder
- C15, C16, C21, C22, C23, C24, C25, C26, C44, C45: footprint Capacitor_SMD:C_0805_2012Metric_Pad1.18x1.45mm_HandSolder -> Capacitor_SMD:C_0603_1608Metric_Pad1.08x0.95mm_HandSolder
- R17, R18, R19, R22, R31, R34, R36: footprint Resistor_SMD:R_0805_2012Metric_Pad1.20x1.40mm_HandSolder -> Resistor_SMD:R_0603_1608Metric_Pad0.98x0.95mm_HandSolder
- R20, R21, R23, R24, R25, R26, R27, R28, R29, R30, R32, R33, R35, R37, R38, R39, R40, R42, R43, R44, R45, R46, R47: footprint Resistor_SMD:R_0805_2012Metric_Pad1.20x1.40mm_HandSolder -> Resistor_SMD:R_0402_1005Metric_Pad0.72x0.64mm_HandSolder
- TP1, TP2, TP3, TP4, TP5: footprint TestPoint:TestPoint_Pad_D2.0mm -> TestPoint:TestPoint_Pad_D1.0mm
Connections:
- net GND: now also Q1.3 (S), Q5.3 (S)
- net at R24.2: now also Q1.2 (G)
- net at R20.2: now also Q5.2 (G)
- net at D1.2 (A), K3.8: now also Q5.1 (D)
- net at D2.2 (A), K1.8: now also Q1.1 (D)
